Commit message: agrega version que muestra brazo robotico

File: brazo_robot_ws/src/brazo_pkg/urdf/brazo.xacro (robot description, xacro)
@@ -1,6 +1,24 @@
 <robot name="brazo_simple">
   <link name="base_link"/>
-  <link name="link1"/>
-  <link name="link2"/>
+  <link name="link1">
+  <visual>
+    <geometry>
+      <box size="0.1 0.1 0.5"/>
+    </geometry>
+    <material name="blue">
+      <color rgba="0 0 1 1"/>
+    </material>
+  </visual>
+</link>
+  <link name="link2">
+  <visual>
+    <geometry>
+      <cylinder length="0.5" radius="0.05"/>
+    </geometry>
+    <material name="red">
+      <color rgba="1 0 0 1"/>
+    </material>
+  </visual>
+</link>
   <joint name="joint1" type="revolute">
     <parent link="base_link"/>
@@ -8,4 +26,5 @@
     <origin xyz="0 0 0.1" rpy="0 0 0"/>
     <axis xyz="0 0 1"/>
+    <limit lower="-1.57" upper="1.57" effort="10" velocity="1"/>
   </joint>
   <joint name="joint2" type="revolute">
@@ -14,4 +33,5 @@
     <origin xyz="0 0 0.5" rpy="0 0 0"/>
     <axis xyz="0 0 1"/>
+    <limit lower="-1.57" upper="1.57" effort="10" velocity="1"/>
   </joint>
 </robot>

Commit message: mueve ambos brazos, movimiento fluido natural

File: brazo_robot_ws/src/brazo_pkg/urdf/brazo.xacro (robot description, xacro)
@@ -14,5 +14,5 @@
   <visual>
     <geometry>
-      <cylinder length="0.5" radius="0.05"/>
+      <box size="0.1 0.1 0.5"/>
     </geometry>
     <material name="red">

Commit message: agrega brazo funcional

File: brazo_robot_ws/src/brazo_pkg/urdf/brazo.xacro (robot description, xacro)
@@ -21,4 +21,26 @@
   </visual>
 </link>
+<link name="wrist">
+  <visual>
+    <geometry>
+      <sphere radius="0.08"/> <!-- bola más grande -->
+    </geometry>
+    <material name="yellow">
+      <color rgba="1 1 0 1"/>
+    </material>
+  </visual>
+</link>
+<link name="link3">
+  <visual>
+    <!-- desplazamos el box 0.15 hacia X para que quede acoplado al borde de la bola -->
+    <origin xyz="0.15 0 0" rpy="0 0 0"/>
+    <geometry>
+      <box size="0.3 0.08 0.08"/> <!-- largo 0.3, delgado en Y,Z -->
+    </geometry>
+    <material name="green">
+      <color rgba="0 1 0 1"/>
+    </material>
+  </visual>
+</link>
   <joint name="joint1" type="revolute">
     <parent link="base_link"/>
@@ -35,3 +57,15 @@
     <limit lower="-1.57" upper="1.57" effort="10" velocity="1"/>
   </joint>
+<joint name="joint_wrist" type="fixed">
+  <parent link="link2"/>
+  <child link="wrist"/>
+  <origin xyz="0 0 0.25" rpy="0 0 0"/> <!-- centro del extremo del brazo rojo -->
+</joint>
+<joint name="joint3" type="revolute">
+  <parent link="wrist"/>
+  <child link="link3"/>
+  <origin xyz="0.08 0 0" rpy="0 0 0"/> <!-- borde de la bola -->
+  <axis xyz="0 1 0"/>
+  <limit lower="-1.57" upper="1.57" effort="10" velocity="1"/>
+</joint>
 </robot>
